File: RPP-Spot-Welder/kicad-pcb-design/spot-welder.kicad_sch (KiCad schematic)
At the start: 18 parts, among them J1 Encoder1, J2 ST7789V Connector, J3 20x4 Connector, J4 100F 16V Super Cap, J5 Weld Pin -, J6 Relay, U1 Pico

Commit message: update the design
Parts:
- removed MOD6: BUCK_CONVERTER, Custom_Modules:BUCK_COVERTER, symbol Custom_Modules:BUCK_CONVERTER
- added MOD6: BOOST_CONVERTER, Custom_Modules:BOOST_COVERTER, symbol Custom_Modules:BOOST_CONVERTER
Connections:
- net +12V: now also MOD6.3 (VOut+)
- net at J4.1 (Pin_1), MOD2.3 (Vout+), MOD5.3 (V+)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: now also MOD6.1 (VIn+)
- net at MOD2.4 (Vout-), MOD5.4 (V-), R1.2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: now also MOD6.2 (VIn-)
- net at MOD7.4 (V-): now also MOD6.4 (VOut-)
Changed lines of the file:
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@@
     (stroke (width 0) (type default))
   )
-  (wire (pts (xy 172.72 34.29) (xy 165.1 34.29))
+  (wire (pts (xy 165.1 34.29) (xy 172.72 34.29))
     (stroke (width 0) (type default))
   )
@@
     (stroke (width 0) (type default))
   )
+  (wire (pts (xy 193.04 39.37) (xy 219.71 39.37))
+    (stroke (width 0) (type default))
+  )
   (wire (pts (xy 285.75 104.14) (xy 274.32 104.14))
     (stroke (width 0) (type default))
@@
     (stroke (width 0) (type default))
   )
+  (wire (pts (xy 193.04 34.29) (xy 204.47 34.29))
+    (stroke (width 0) (type default))
+  )
   (wire (pts (xy 262.89 137.16) (xy 262.89 201.93))
     (stroke (width 0) (type default))
@@
     (stroke (width 0) (type default))
   )
-  (wire (pts (xy 193.04 34.29) (xy 204.47 34.29))
-    (stroke (width 0) (type default))
-  )
   (wire (pts (xy 224.79 201.93) (xy 242.57 201.93))
     (stroke (width 0) (type default))
@@
   )
   (wire (pts (xy 242.57 201.93) (xy 262.89 201.93))
-    (stroke (width 0) (type default))
-  )
-  (wire (pts (xy 193.04 39.37) (xy 219.71 39.37))
     (stroke (width 0) (type default))
   )
@@
         (path "/c006826f-e3dc-4ff5-8da7-c42a0a9fadb3"
           (reference "J1") (unit 1)
-        )
-      )
-    )
-  )
-  (symbol (lib_id "Custom_Modules:BUCK_CONVERTER") (at 182.88 36.83 0) (unit 1)
-    (in_bom yes) (on_board yes) (dnp no) (fields_autoplaced)
-    (property "Reference" "MOD6" (at 182.88 29.21 0)
-      (effects (font (size 1.27 1.27)))
-    )
-    (property "Value" "BUCK_CONVERTER" (at 182.88 31.75 0)
-      (effects (font (size 1.27 1.27)))
-    )
-    (property "Footprint" "Custom_Modules:BUCK_COVERTER" (at 180.34 36.83 0)
-      (effects (font (size 1.27 1.27)) hide)
-    )
-    (property "Datasheet" "" (at 180.34 36.83 0)
-      (effects (font (size 1.27 1.27)) hide)
-    )
-    (pin "1")
-    (pin "2")
-    (pin "3")
-    (pin "4")
-    (instances
-      (project "spot-welder"
-        (path "/c006826f-e3dc-4ff5-8da7-c42a0a9fadb3"
-          (reference "MOD6") (unit 1)
         )
       )
@@
         )
       )
+    )
+  )
+  (symbol (lib_id "Custom_Modules:BOOST_CONVERTER") (at 182.88 36.83 0) (unit 1)
+    (in_bom yes) (on_board yes) (dnp no) (fields_autoplaced)
+    (property "Reference" "MOD6" (at 182.88 29.21 0)
+      (effects (font (size 1.27 1.27)))
+    )
+    (property "Value" "BOOST_CONVERTER" (at 182.88 31.75 0)
+      (effects (font (size 1.27 1.27)))
+    )
+    (property "Footprint" "Custom_Modules:BOOST_COVERTER" (at 180.34 36.83 0)
+      (effects (font (size 1.27 1.27)) hide)
+    )
+    (property "Datasheet" "" (at 180.34 36.83 0)
+      (effects (font (size 1.27 1.27)) hide)
+    )
+    (pin "1")
+    (pin "2")
+    (pin "3")
+    (pin "4")
+    (instances
+      (project "spot-welder"
+        (path "/c006826f-e3dc-4ff5-8da7-c42a0a9fadb3"
+          (reference "MOD6") (unit 1)
+        )
+      )

Commit message: update the schmatic
Connections:
- net VCC: now also MOD6.1 (VIn+)
- net at J4.1 (Pin_1), MOD2.3 (Vout+), MOD5.3 (V+)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: no longer MOD6.1 (VIn+)
- net at MOD2.4 (Vout-), MOD5.4 (V-), R1.2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: no longer MOD6.2 (VIn-)
- net at MOD2.2 (Vin-), MOD3.5 (Load): now also MOD6.2 (VIn-)
Changed lines of the file:
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@@
   (junction (at 152.4 139.7) (diameter 0) (color 0 0 0 0)
   )
-  (junction (at 165.1 77.47) (diameter 0) (color 0 0 0 0)
-  )
   (junction (at 87.63 134.62) (diameter 0) (color 0 0 0 0)
   )
@@
   (junction (at 87.63 128.27) (diameter 0) (color 0 0 0 0)
   )
+  (junction (at 99.06 86.36) (diameter 0) (color 0 0 0 0)
+  )
   (junction (at 224.79 201.93) (diameter 0) (color 0 0 0 0)
   )
@@
   )
   (junction (at 262.89 201.93) (diameter 0) (color 0 0 0 0)
-  )
-  (junction (at 167.64 86.36) (diameter 0) (color 0 0 0 0)
   )
   (no_connect (at 166.37 172.72))
@@
     (stroke (width 0) (type default))
   )
+  (wire (pts (xy 99.06 39.37) (xy 99.06 86.36))
+    (stroke (width 0) (type default))
+  )
   (wire (pts (xy 204.47 34.29) (xy 227.33 34.29))
     (stroke (width 0) (type default))
@@
     (stroke (width 0) (type default))
   )
+  (wire (pts (xy 99.06 39.37) (xy 172.72 39.37))
+    (stroke (width 0) (type default))
+  )
   (wire (pts (xy 87.63 162.56) (xy 96.52 162.56))
     (stroke (width 0) (type default))
@@
     (stroke (width 0) (type default))
   )
-  (wire (pts (xy 167.64 39.37) (xy 172.72 39.37))
-    (stroke (width 0) (type default))
-  )
   (wire (pts (xy 224.79 214.63) (xy 224.79 201.93))
     (stroke (width 0) (type default))
@@
     (stroke (width 0) (type default))
   )
-  (wire (pts (xy 167.64 86.36) (xy 236.22 86.36))
-    (stroke (width 0) (type default))
-  )
-  (wire (pts (xy 167.64 86.36) (xy 167.64 39.37))
-    (stroke (width 0) (type default))
-  )
   (wire (pts (xy 274.32 92.71) (xy 274.32 95.25))
     (stroke (width 0) (type default))
@@
     (stroke (width 0) (type default))
   )
+  (wire (pts (xy 93.98 34.29) (xy 93.98 77.47))
+    (stroke (width 0) (type default))
+  )
   (wire (pts (xy 274.32 114.3) (xy 236.22 114.3))
     (stroke (width 0) (type default))
@@
     (stroke (width 0) (type default))
   )
-  (wire (pts (xy 153.67 86.36) (xy 167.64 86.36))
+  (wire (pts (xy 153.67 86.36) (xy 236.22 86.36))
     (stroke (width 0) (type default))
   )
@@
     (stroke (width 0) (type default))
   )
-  (wire (pts (xy 165.1 34.29) (xy 172.72 34.29))
-    (stroke (width 0) (type default))
-  )
   (wire (pts (xy 166.37 142.24) (xy 110.49 142.24))
     (stroke (width 0) (type default))
@@
     (stroke (width 0) (type default))
   )
-  (wire (pts (xy 161.29 77.47) (xy 165.1 77.47))
+  (wire (pts (xy 161.29 77.47) (xy 267.97 77.47))
     (stroke (width 0) (type default))
   )
@@
     (stroke (width 0) (type default))
   )
-  (wire (pts (xy 165.1 34.29) (xy 165.1 77.47))
-    (stroke (width 0) (type default))
-  )
   (wire (pts (xy 166.37 144.78) (xy 160.02 144.78))
     (stroke (width 0) (type default))
@@
     (stroke (width 0) (type default))
   )
+  (wire (pts (xy 93.98 34.29) (xy 172.72 34.29))
+    (stroke (width 0) (type default))
+  )
   (wire (pts (xy 262.89 137.16) (xy 262.89 201.93))
     (stroke (width 0) (type default))
@@
     (stroke (width 0) (type default))
   )
-  (wire (pts (xy 165.1 77.47) (xy 267.97 77.47))
-    (stroke (width 0) (type default))
-  )
